Commit message: Update robot_core.xacro

File: description/robot_core.xacro (robot description, xacro)
@@ -1,6 +1,80 @@
 <?xml version="1.0"?>
-<robot xmlns:xacro="http://www.ros.org/wiki/xacro" >
-<!-- BASE LINK -->
-    <link name="base_link">
-    </link>
+<robot xmlns:xacro="http://www.ros.org/wiki/xacro">
+<link name="base_link">
+</link>
+<joint name="chassis_joint" type="fixed">
+    <parent link="base_link"/>
+    <child link="chassis"/>
+    <origin xyz="-0.2 0 0"/>
+</joint>
+<link name="chassis">
+    <visual>
+        <origin xyz="0.2 0 0.2" rpy="0 0 0"/>
+        <geometry>
+            <box size="0.4 0.4 0.4"/>
+        </geometry>
+    </visual>
+    <collision>
+        <origin xyz="0.2 0 0.2" rpy="0 0 0"/>
+        <geometry>
+            <box size="0.4 0.4 0.4"/>
+        </geometry>
+    </collision>
+</link>
+<!-- LEFT FRONT WHEEL -->
+<joint name="left_front_wheel_joint" type="continuous">
+    <parent link="base_link"/>
+    <child link="left_front_wheel"/>
+    <origin xyz="0.15 0.2 0" rpy="-${pi/2} 0 0"/>
+    <axis xyz="0 0 1"/>
+</joint>
+<link name="left_front_wheel">
+    <visual>
+        <geometry>
+            <cylinder length="0.04" radius="0.05" />/>
+        </geometry>
+    </visual>
+</link>
+<!-- LEFT BACK WHEEL -->
+<joint name="left_back_wheel_joint" type="continuous">
+    <parent link="base_link"/>
+    <child link="left_back_wheel"/>
+    <origin xyz="-0.15 0.2 0" rpy="-${pi/2} 0 0"/>
+    <axis xyz="0 0 1"/>
+</joint>
+<link name="left_back_wheel">
+    <visual>
+        <geometry>
+            <cylinder length="0.04" radius="0.05" />/>
+        </geometry>
+    </visual>
+</link>
+<!-- RIGHT FRONT WHEEL -->
+<joint name="right_front_wheel_joint" type="continuous">
+    <parent link="base_link"/>
+    <child link="right_front_wheel"/>
+    <origin xyz="0.15 -0.2 0" rpy="${pi/2} 0 0"/>
+    <axis xyz="0 0 -1"/>
+</joint>
+<link name="right_front_wheel">
+    <visual>
+        <geometry>
+            <cylinder length="0.04" radius="0.05" />/>
+        </geometry>
+    </visual>
+</link>
+<!-- RIGHT FRONT WHEEL -->
+<joint name="right_back_wheel_joint" type="continuous">
+    <parent link="base_link"/>
+    <child link="right_back_wheel"/>
+    <origin xyz="-0.15 -0.2 0" rpy="${pi/2} 0 0"/>
+    <axis xyz="0 0 -1"/>
+</joint>
+<link name="right_back_wheel">
+    <visual>
+        <geometry>
+            <cylinder length="0.04" radius="0.05" />/>
+        </geometry>
+    </visual>
+</link>
 </robot>
